File: hardware/swadge2019.sch (KiCad schematic (older format))
At the start: 18 parts, among them SW1 TACTILE, SW2 TACTILE, SW3 TACTILE, SW4 TACTILE, SW5 TACTILE, SW6 TACTILE

Commit message: bump design
Parts:
- added C1, C3: 10u, C_0805, symbol C
- added C2: 1u, C_0805, symbol C
- added R3: 22k, R_0805, symbol R
- added R4, R7: 47k, R_0805, symbol R
- added R5: 220k, R_0805, symbol R
- added R6, R8: 10k, R_0805, symbol R
- R1: value R -> 10k
- R2: value R -> NOPOP-internal?
- gave numbers to parts that had none: 3
Connections:
- net ADCBIN is gone; now on net ADCPIN: ESP1.2 (ADC)
- net +3V3: now also C1.1
- net GND: now also U1.2 (Vss), C1.2, C3.2, R8.2
- net AUDPWR: now reaches ESP1.6 (GPIO12)
- net AUDPWR: now also U1.5 (Vdd), C3.1, R6.1, R7.1
- net ADCPIN: now reaches U1.1 (Vout)
- net ADCPIN: now also R5.1
- net VGS: now reaches U1.3 (Vin+)
- net VGS: now also R4.1, R7.2, R8.1
- net at U1.4 (Vin-): now also R3.1, R5.2
- net at Y1.1: now also C2.2, R6.2
- new net: C2.1, R3.2, R4.2
Other:
- note added: "During colorchord operations, turn on GPIO12."
- note added: "GPIO15 may be used as an additional input if an external pull-down resistor is applied."
- moved on the sheet: U1

Commit message: update swadge set
Parts:
- removed D1, D2, D3, D4, D5, D6: WS2813, WS2813, symbol WS2813
- removed P1: CONN_01X04, symbol CONN_01X04
- removed SW5, SW6: TACTILE, TACTILE10, symbol TACTILE
- added BT1, BT2: Battery, BCAAPC, symbol Battery
- added C4: .1u, C_0805, symbol C
- added D1, D2, D3, D4, D5, D6: SK6812SIDE, SK6812SIDE, symbol SK6812SIDE
- added P1: PGM, Pin_Header_Straight_1x05, symbol CONN_01X05
- added P2: USBMicroB-10118194-0001LF, USBMicroB-10118194-0001LF, symbol USBMicroB-10118194-0001LF
- added P3, P4, P5, P6: CONN_1, 632HOLE, symbol CONN_1
- added SW7: SWITCH_INV, JS_SWITCH, symbol SWITCH_INV
- added U2: AP1117SOT223, SOT-223, symbol AP1117SOT223
- U1: footprint (none) -> SOT-23-5
- Y1: footprint CP_Radial_D10.0mm_P2.50mm_P5.00mm -> C_Radial_D8_L13_P3.8
Connections:
- net +3V3: now also C4.1, D1.2 (VDD), D2.2 (VDD), D3.2 (VDD), D4.2 (VDD), D5.2 (VDD), D6.2 (VDD), SW7.2
- net GND: now also BT2.2, C4.2, D1.4 (GND), D2.4 (GND), D3.4 (GND), D4.4 (GND), D5.4 (GND), D6.4 (GND), P1.1 (P1), P2.5 (GND), P2.6 (CASE), P2.7 (CASE), P2.8 (CASE), P2.9 (CASE), P3.1, P4.1, P5.1, P6.1, U2.1 (GND)
- net GPIO0: now also P1.5 (P5)
- net RX: now also D1.1 (DIN), P1.2 (P2)
- net TX: now also P1.3 (P3)
- net GPIO14: no longer names the net of ESP1.5 (GPIO14)
- new net: D1.3 (DOUT), D2.1 (DIN)
- new net: D2.3 (DOUT), D3.1 (DIN)
- new net: D3.3 (DOUT), D4.1 (DIN)
- new net: D4.3 (DOUT), D5.1 (DIN)
- new net: D5.3 (DOUT), D6.1 (DIN)
- new net: BT1.1, SW7.1
- new net: SW7.3, U2.2 (Vout), U2.4 (Vout2)
- new net: BT1.2, BT2.1
- new net +5V: P1.4 (P4), P2.1 (VCC), U2.3 (Vin)

Commit message: bump design
Parts:
- added C5, C6: .1u, C_0805, symbol C
- added P10, P11, P12, P13, P7, P8, P9: CONN_1, 632HOLE, symbol CONN_1
Connections:
- net +3V3: now also C5.1
- net +5V: now also C6.1
- net AUDPWR: now also ESP1.5 (GPIO14); no longer ESP1.6 (GPIO12)
- net GND: now also C5.2, C6.2, P10.1, P11.1, P12.1, P13.1, P7.1, P8.1, P9.1
- net GPIO13: now also P2.3 (D+)
- net GPIO12: now reaches P2.2 (D-)
- net GPIO12: now also ESP1.6 (GPIO12)
Changed lines of the file:
@@
 	1    0    0    -1
 $EndComp
-Text GLabel 3150 2300 0    60   Input ~ 0
+Text GLabel 3150 2200 0    60   Input ~ 0
 AUDPWR
 Text GLabel 800  2000 1    60   Input ~ 0
@@
 	0    -1   -1   0
 $EndComp
+$Comp
+L C C5
+U 1 1 5B94AF8F
+P 7750 3150
+F 0 "C5" H 7775 3250 50  0000 L CNN
+F 1 ".1u" H 7775 3050 50  0000 L CNN
+F 2 "C_0805" H 7788 3000 50  0000 C CNN
+F 3 "" H 7750 3150 50  0000 C CNN
+	1    7750 3150
+	1    0    0    -1
+$EndComp
+$Comp
+L GND #PWR047
+U 1 1 5B94AF95
+P 7750 3300
+F 0 "#PWR047" H 7750 3050 50  0001 C CNN
+F 1 "GND" H 7750 3150 50  0000 C CNN
+F 2 "" H 7750 3300 50  0000 C CNN
+F 3 "" H 7750 3300 50  0000 C CNN
+	1    7750 3300
+	1    0    0    -1
+$EndComp
+$Comp
+L +3.3V #PWR048
+U 1 1 5B94AF9B
+P 7750 3000
+F 0 "#PWR048" H 7750 2850 50  0001 C CNN
+F 1 "+3.3V" H 7750 3140 50  0000 C CNN
+F 2 "" H 7750 3000 50  0000 C CNN
+F 3 "" H 7750 3000 50  0000 C CNN
+	1    7750 3000
+	1    0    0    -1
+$EndComp
+$Comp
+L CONN_1 P10
+U 1 1 5B94B412
+P 5500 4200
+F 0 "P10" H 5580 4200 40  0000 L CNN
+F 1 "CONN_1" H 5500 4255 30  0001 C CNN
+F 2 "632HOLE" H 5500 4200 60  0000 C CNN
+F 3 "" H 5500 4200 60  0000 C CNN
+	1    5500 4200
+	-1   0    0    1
+$EndComp
+$Comp
+L CONN_1 P9
+U 1 1 5B94B418
+P 5500 4050
+F 0 "P9" H 5580 4050 40  0000 L CNN
+F 1 "CONN_1" H 5500 4105 30  0001 C CNN
+F 2 "632HOLE" H 5500 4050 60  0000 C CNN
+F 3 "" H 5500 4050 60  0000 C CNN
+	1    5500 4050
+	-1   0    0    1
+$EndComp
+$Comp
+L CONN_1 P8
+U 1 1 5B94B41E
+P 5500 3900
+F 0 "P8" H 5580 3900 40  0000 L CNN
+F 1 "CONN_1" H 5500 3955 30  0001 C CNN
+F 2 "632HOLE" H 5500 3900 60  0000 C CNN
+F 3 "" H 5500 3900 60  0000 C CNN
+	1    5500 3900
+	-1   0    0    1
+$EndComp
+$Comp
+L CONN_1 P7
+U 1 1 5B94B424
+P 5500 3750
+F 0 "P7" H 5580 3750 40  0000 L CNN
+F 1 "CONN_1" H 5500 3805 30  0001 C CNN
+F 2 "632HOLE" H 5500 3750 60  0000 C CNN
+F 3 "" H 5500 3750 60  0000 C CNN
+	1    5500 3750
+	-1   0    0    1
+$EndComp
+$Comp
+L GND #PWR049
+U 1 1 5B94B42A
+P 5650 3750
+F 0 "#PWR049" H 5650 3500 50  0001 C CNN
+F 1 "GND" H 5650 3600 50  0000 C CNN
+F 2 "" H 5650 3750 50  0000 C CNN
+F 3 "" H 5650 3750 50  0000 C CNN
+	1    5650 3750
+	0    -1   -1   0
+$EndComp
+$Comp
+L GND #PWR050
+U 1 1 5B94B430
+P 5650 3900
+F 0 "#PWR050" H 5650 3650 50  0001 C CNN
+F 1 "GND" H 5650 3750 50  0000 C CNN
+F 2 "" H 5650 3900 50  0000 C CNN
+F 3 "" H 5650 3900 50  0000 C CNN
+	1    5650 3900
+	0    -1   -1   0
+$EndComp
+$Comp
+L GND #PWR051
+U 1 1 5B94B436
+P 5650 4050
+F 0 "#PWR051" H 5650 3800 50  0001 C CNN
+F 1 "GND" H 5650 3900 50  0000 C CNN
+F 2 "" H 5650 4050 50  0000 C CNN
+F 3 "" H 5650 4050 50  0000 C CNN
+	1    5650 4050
+	0    -1   -1   0
+$EndComp
+$Comp
+L GND #PWR052
+U 1 1 5B94B43C
+P 5650 4200
+F 0 "#PWR052" H 5650 3950 50  0001 C CNN
+F 1 "GND" H 5650 4050 50  0000 C CNN
+F 2 "" H 5650 4200 50  0000 C CNN
+F 3 "" H 5650 4200 50  0000 C CNN
+	1    5650 4200
+	0    -1   -1   0
+$EndComp
+$Comp
+L CONN_1 P12
+U 1 1 5B94B51E
+P 5500 4500
+F 0 "P12" H 5580 4500 40  0000 L CNN
+F 1 "CONN_1" H 5500 4555 30  0001 C CNN
+F 2 "632HOLE" H 5500 4500 60  0000 C CNN
+F 3 "" H 5500 4500 60  0000 C CNN
+	1    5500 4500
+	-1   0    0    1
+$EndComp
+$Comp
+L CONN_1 P11
+U 1 1 5B94B524
+P 5500 4350
+F 0 "P11" H 5580 4350 40  0000 L CNN
+F 1 "CONN_1" H 5500 4405 30  0001 C CNN
+F 2 "632HOLE" H 5500 4350 60  0000 C CNN
+F 3 "" H 5500 4350 60  0000 C CNN
+	1    5500 4350
+	-1   0    0    1
+$EndComp
+$Comp
+L GND #PWR053
+U 1 1 5B94B52A
+P 5650 4350
+F 0 "#PWR053" H 5650 4100 50  0001 C CNN
+F 1 "GND" H 5650 4200 50  0000 C CNN
+F 2 "" H 5650 4350 50  0000 C CNN
+F 3 "" H 5650 4350 50  0000 C CNN
+	1    5650 4350
+	0    -1   -1   0
+$EndComp
+$Comp
+L GND #PWR054
+U 1 1 5B94B530
+P 5650 4500
+F 0 "#PWR054" H 5650 4250 50  0001 C CNN
+F 1 "GND" H 5650 4350 50  0000 C CNN
+F 2 "" H 5650 4500 50  0000 C CNN
+F 3 "" H 5650 4500 50  0000 C CNN
+	1    5650 4500
+	0    -1   -1   0
+$EndComp
+$Comp
+L CONN_1 P13
+U 1 1 5B94B7A5
+P 4700 3600
+F 0 "P13" H 4780 3600 40  0000 L CNN
+F 1 "CONN_1" H 4700 3655 30  0001 C CNN
+F 2 "632HOLE" H 4700 3600 60  0000 C CNN
+F 3 "" H 4700 3600 60  0000 C CNN
+	1    4700 3600
+	-1   0    0    1
+$EndComp
+$Comp
+L GND #PWR055
+U 1 1 5B94B7AB
+P 4850 3600
+F 0 "#PWR055" H 4850 3350 50  0001 C CNN
+F 1 "GND" H 4850 3450 50  0000 C CNN
+F 2 "" H 4850 3600 50  0000 C CNN
+F 3 "" H 4850 3600 50  0000 C CNN
+	1    4850 3600
+	0    -1   -1   0
+$EndComp
+$Comp
+L C C6
+U 1 1 5B94B980
+P 6550 3150
+F 0 "C6" H 6575 3250 50  0000 L CNN
+F 1 ".1u" H 6575 3050 50  0000 L CNN
+F 2 "C_0805" H 6588 3000 50  0000 C CNN
+F 3 "" H 6550 3150 50  0000 C CNN
+	1    6550 3150
+	1    0    0    -1
+$EndComp
+$Comp
+L GND #PWR056
+U 1 1 5B94B986
+P 6550 3300
+F 0 "#PWR056" H 6550 3050 50  0001 C CNN
+F 1 "GND" H 6550 3150 50  0000 C CNN
+F 2 "" H 6550 3300 50  0000 C CNN
+F 3 "" H 6550 3300 50  0000 C CNN
+	1    6550 3300
+	1    0    0    -1
+$EndComp
+$Comp
+L +5V #PWR057
+U 1 1 5B94BD38
+P 6550 3000
+F 0 "#PWR057" H 6550 2850 50  0001 C CNN
+F 1 "+5V" H 6550 3140 50  0000 C CNN
+F 2 "" H 6550 3000 50  0000 C CNN
+F 3 "" H 6550 3000 50  0000 C CNN
+	1    6550 3000
+	1    0    0    -1
+$EndComp
+Text GLabel 3150 2300 0    60   Input ~ 0
+GPIO12
+Text GLabel 7150 4400 0    60   Input ~ 0
+GPIO12
+Text GLabel 7150 4500 0    60   Input ~ 0
+GPIO13
 $EndSCHEMATC

Commit message: update for gerbers for productio
Parts:
- added R9: 1.5k, R_0805, symbol R
Connections:
- net +3V3: now also R9.1
- net GPIO12: now also R9.2

Commit message: bump design a little...
Parts:
- SW7: Cost100 (none) -> 0.48010; Digikey (none) -> 401-1999-6-ND

Commit message: Bump design
Parts:
- removed P3, P4, P5, P6: CONN_1, 632HOLE, symbol CONN_1
- removed SW2, SW3: TACTILE, TACTILE10, symbol TACTILE
- added C7, C8: .1u, C_0805, symbol C
- added P3: SAO, Pin_Header_Straight_2x02, symbol CONN_02X02
- added R10: 1k, R_0805, symbol R
- added R11: 1.5k, R_0805, symbol R
- added SW3: MODE, TACT_3x6_SINGLE, symbol SPST
- C3: value 10u -> 22u
- P2: value USBMicroB-10118194-0001LF -> USBMicroB-10118192-0001LF; footprint USBMicroB-10118194-0001LF -> USBMicroB-10118192-0001LF
- SW1: value TACTILE -> B
- SW2: renamed from SW4; value TACTILE -> A
- Y1: value Microphone -> Mic
Connections:
- net +3V3: now also C8.1, P3.1 (P1), R11.1
- net AUDPWR: now also C7.1, R10.2; no longer ESP1.5 (GPIO14)
- net GND: now also C7.2, C8.2, P3.2 (P2), SW3.2
- net GPIO0: now also SW3.1
- net GPIO12: no longer P2.2 (D-), R9.2
- net GPIO13: now also SW2.1; no longer P2.3 (D+)
- net GPIO4: now also R9.2, P3.3 (P3); no longer SW2.1
- net GPIO5: now also P3.4 (P4), R11.2
- new net: ESP1.5 (GPIO14), R10.1

Commit message: bump all
Parts:
- added P4: CONN_1, round_suncats_half, symbol CONN_1
Changed lines of the file:
@@
 	1    0    0    -1
 $EndComp
+$Comp
+L CONN_1 P4
+U 1 1 5BC40676
+P 8900 6000
+F 0 "P4" H 8980 6000 40  0000 L CNN
+F 1 "CONN_1" H 8900 6055 30  0001 C CNN
+F 2 "round_suncats_half" H 8900 6000 60  0000 C CNN
+F 3 "" H 8900 6000 60  0000 C CNN
+	1    8900 6000
+	-1   0    0    1
+$EndComp
 $EndSCHEMATC

Commit message: Bump
Parts:
- added P5: ~, front_silkscreen, symbol CONN_1
- added P6: CONN_1, round_suncats_half_mask, symbol CONN_1
Changed lines of the file:
@@
+	-1   0    0    1
+$EndComp
+$Comp
+L CONN_1 P5
+U 1 1 5BC40D15
+P 8900 6150
+F 0 "P5" H 8980 6150 40  0000 L CNN
+F 1 "~" H 8900 6205 30  0001 C CNN
+F 2 "front_silkscreen" H 8900 6150 60  0000 C CNN
+F 3 "" H 8900 6150 60  0000 C CNN
+	1    8900 6150
+	-1   0    0    1
+$EndComp
+$Comp
+L CONN_1 P6
+U 1 1 5BC41066
+P 8900 5850
+F 0 "P6" H 8980 5850 40  0000 L CNN
+F 1 "CONN_1" H 8900 5905 30  0001 C CNN
+F 2 "round_suncats_half_mask" H 8900 5850 60  0000 C CNN
+F 3 "" H 8900 5850 60  0000 C CNN
+	1    8900 5850
 	-1   0    0    1
 $EndComp
