File: hardware/swadge2019.kicad_pcb (KiCad board)
At the start: 2 copper layers, 78.9 x 76.6 mm, 45 parts, among them P1 PGM, P10 CONN_1, P11 CONN_1, P12 CONN_1, P13 CONN_1, P2 USBMicroB-10118194-0001LF, P3 CONN_1, P4 CONN_1, P5 CONN_1, P6 CONN_1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

Commit message: bump design a little...
Parts:
- D1, D4: footprint SK6812SIDE -> charles:SK6812SIDE
- D2: renamed from D6; footprint SK6812SIDE -> charles:SK6812SIDE
- D3: renamed from D5; footprint SK6812SIDE -> charles:SK6812SIDE
- D5: renamed from D3; footprint SK6812SIDE -> charles:SK6812SIDE
- D6: renamed from D2; footprint SK6812SIDE -> charles:SK6812SIDE
- moved P1 3.92 mm to (95.1, 37.0), turned to 270 degrees
- moved D5 0.28 mm to (107.8, 68.0), turned to 60 degrees
- moved D3 0.25 mm to (65.8, 68.5), turned to 300 degrees
- moved D4 0.17 mm to (86.8, 80.0), turned to 0 degrees
- moved D6 0.14 mm to (108.3, 42.5), turned to 120 degrees
- moved D2 0.13 mm to (64.8, 42.5), turned to 240 degrees
- moved D1 0.10 mm to (86.3, 30.0), turned to 180 degrees
Connections:
- D2 pad 1: Net-(D5-Pad3) -> Net-(D1-Pad3)
- D2 pad 3: (no net) -> Net-(D2-Pad3)
- D3 pad 1: Net-(D4-Pad3) -> Net-(D2-Pad3)
- D3 pad 3: Net-(D5-Pad3) -> Net-(D3-Pad3)
- D5 pad 1: Net-(D2-Pad3) -> Net-(D4-Pad3)
- D5 pad 3: Net-(D3-Pad3) -> Net-(D5-Pad3)
- D6 pad 1: Net-(D1-Pad3) -> Net-(D5-Pad3)
- D6 pad 3: Net-(D2-Pad3) -> (no net)
Routing:
- net Net-(BT1-Pad1): track 54.1 -> 109.3 mm, vias 1 -> 2
- net +3V3: track 224.8 -> 245.0 mm, vias 15 -> 14
- net GPIO0: track 36.8 -> 51.1 mm, vias 3 -> 5
- net GND: track 328.3 -> 320.6 mm, vias 25 -> 26
- net +5V: track 106.6 -> 113.2 mm
- net TX: track 6.54 -> 11.4 mm
- net RX: track 33.6 -> 29.5 mm
- net Net-(D1-Pad3): track 28.6 -> 32.1 mm, vias 2 -> 0
- net Net-(D4-Pad3): track 25.1 -> 28.0 mm, vias 0 -> 2
- net (no net): track 15.8 -> 13.0 mm, vias 1 -> 0
- net Net-(D3-Pad3): track 26.5 -> 29.2 mm, vias 2 -> 0
- net Net-(D5-Pad3): track 26.8 -> 25.6 mm
- net Net-(D2-Pad3): track 25.7 -> 27.0 mm

Commit message: bump
Parts:
- moved SW3 0.50 mm to (109.8, 55.1)
- moved SW2 0.50 mm to (63.2, 55.1)
Routing:
- net +5V: track 113.2 -> 81.5 mm, vias 4 -> 2
- net GND: track 320.6 -> 328.0 mm, vias 26 -> 27
- net +3V3: track 245.0 -> 249.5 mm, vias 14 -> 12
- net Net-(D4-Pad3): track 28.0 -> 25.3 mm
- net Net-(D3-Pad3): track 29.2 -> 26.8 mm
- net Net-(D1-Pad3): track 32.1 -> 33.2 mm
Other:
- board text added: "GND RX TX +5V G0"
- board text added: "SWADGE2019 REV A Hi, Nick."
- board text removed: "SWADGE2019 REV - Hi, Nick."

Commit message: Bump design
Parts:
- removed P4, P5, P6: CONN_1, 632HOLE
- removed SW4: TACTILE, TACTILE10
- added C7: .1u, C_0805, F.Cu at (58.6, 78.5)
- added C8: .1u, C_0805, F.Cu at (69.8, 102.5)
- added R10: 1k, R_0805, F.Cu at (63.6, 71.3)
- added R11: 1.5k, R_0805, F.Cu at (98.6, 81.9)
- C3: value 10u -> 22u
- P2: value USBMicroB-10118194-0001LF -> USBMicroB-10118192-0001LF; footprint USBMicroB-10118194-0001LF -> USBMicroB-10118192-0001LF
- P3: value CONN_1 -> SAO; footprint 632HOLE -> Pin_Header_Straight_2x02
- SW1: value TACTILE -> B
- SW2: value TACTILE -> A
- SW3: value TACTILE -> MODE; footprint TACTILE10 -> TACT_3x6_SINGLE
- Y1: value Microphone -> Mic
- moved P3 51.1 mm to (97.9, 75.8)
- moved SW3 41.4 mm to (76.3, 79.3), turned to 180 degrees
- moved SW2 40.6 mm to (64.6, 95.7), turned to 150 degrees
- moved R1 36.6 mm to (86.9, 79.0), turned to 145 degrees
- moved P2 34.5 mm to (61.5, 126.4)
- moved C5 33.8 mm to (50.2, 77.0), turned to 90 degrees
- moved U2 32.2 mm to (75.7, 97.4), turned to 0 degrees
- moved D4 31.5 mm to (76.1, 109.6)
- moved D3 30.5 mm to (47.3, 92.8)
- moved SW7 28.0 mm to (90.7, 121.8)
- moved Y1 26.1 mm to (70.4, 87.2), turned to 320 degrees
- moved D5 25.0 mm to (105.1, 92.9)
- moved R9 24.9 mm to (94.4, 77.3), turned to 270 degrees
- moved D2 24.4 mm to (47.3, 59.5)
- moved R2 24.0 mm to (91.6, 86.9)
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Connections:
- ESP1 pad 5: AUDPWR -> Net-(ESP1-Pad5)
- ESP1 pad 6: GPIO12 -> (no net)
- P2 pad 2: GPIO12 -> (no net)
- P2 pad 3: GPIO13 -> (no net)
- P3 pad 1: GND -> +3V3
- R9 pad 2: GPIO12 -> GPIO4
- SW2 pad 1: GPIO0 -> GPIO13
- SW3 pad 1: GPIO5 -> GPIO0
- SW3 pad 2: (no net) -> GND
Routing:
- net +3V3: track 249.5 -> 409.4 mm, vias 12 -> 16
- net GND: track 328.0 -> 216.2 mm, vias 27 -> 19
- net Net-(BT1-Pad1): track 109.0 -> 176.8 mm
- net GPIO12: track 48.2 -> 0.00 mm, vias 2 -> 0
- net Net-(SW7-Pad3): track 30.8 -> 66.3 mm, vias 1 -> 4
- net Net-(BT1-Pad2): track 16.3 -> 50.4 mm
- net GPIO4: track 47.3 -> 24.1 mm, vias 0 -> 1
- net Net-(D5-Pad3): track 25.6 -> 40.1 mm
- net Net-(D2-Pad3): track 27.0 -> 39.4 mm
- net GPIO13: track 42.8 -> 32.0 mm, vias 1 -> 2
- net GPIO5: track 23.0 -> 31.3 mm, vias 0 -> 1
- net Net-(D4-Pad3): track 25.3 -> 31.8 mm
- net Net-(D3-Pad3): track 26.8 -> 32.2 mm
- net Net-(ESP1-Pad5): track 0.00 -> 5.31 mm
- net GPIO2: track 27.2 -> 31.7 mm
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Other:
- board size 78.9 x 76.6 mm -> 100 x 95.3 mm
- board text added: "SWADGE2019 REV B Hi, Deb"
- board text removed: "SWADGE2019 REV A Hi, Nick."

Commit message: bump all
Parts:
- added G***: LOGO, LOGO, F.Cu at (93.6, 64.7)
- added G***: LOGO, LOGO, B.Cu at (76.8, 48.2)
- added G***: LOGO, LOGO, B.Cu at (76.2, 105.8)
- added G***: LOGO, LOGO, B.Cu at (76.2, 105.7)
- added P5: ~, LOGO, F.Cu at (76.0, 75.2)
Routing:
- net +3V3: track 409.4 -> 410.7 mm
- net Net-(D5-Pad3): track 40.1 -> 39.0 mm
Other:
- board text added: "SWADGE2019 REV B All Aircraft Report"
- board text removed: "SWADGE2019 REV B Hi, Deb"

Commit message: Bump
Other:
- board text added: "BAT"
- board text added: "Made in China"
- board text added: "USB"
Changed lines of the file:
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@@
     (links 96)
     (no_connects 0)
-    (area 26.149999 32.848729 126.250001 128.211525)
+    (area 17.593375 24.188475 134.806625 132.340001)
     (thickness 1.6)
-    (drawings 113)
+    (drawings 116)
     (tracks 489)
     (zones 0)
@@
       (drillshape 0)
       (scaleselection 1)
-      (outputdirectory swadge2019-revA))
+      (outputdirectory swadge2019-revB))
   )
   (net 0 "")
@@
       (effects (font (size 1 1) (thickness 0.15)) (justify mirror))
     )
-    (fp_text value SWITCH_INV (at 0 -2 180) (layer B.SilkS)
+    (fp_text value SWITCH_INV (at 0.59 4.92 180) (layer B.SilkS)
       (effects (font (size 1 1) (thickness 0.15)) (justify mirror))
     )
@@
     )
   )
+  (gr_text BAT (at 97.08 126.18) (layer B.SilkS)
+    (effects (font (size 1.5 1.5) (thickness 0.3)) (justify mirror))
+  )
+  (gr_text USB (at 83.93 126.18) (layer B.SilkS)
+    (effects (font (size 1.5 1.5) (thickness 0.3)) (justify mirror))
+  )
+  (gr_text "Made in China" (at 74.63 79.38) (layer B.SilkS)
+    (effects (font (size 1.5 1.5) (thickness 0.3)) (justify mirror))
+  )
   (gr_circle (center 96.14 73.8) (end 96.51 73.82) (layer F.SilkS) (width 0.15))

Commit message: Bump
Routing:
- net Net-(BT1-Pad1): track 176.8 -> 185.4 mm
- net Net-(BT1-Pad2): track 50.4 -> 51.8 mm
- net GND: track 216.2 -> 217.4 mm

Commit message: update design
Parts:
- C1: value 10u -> 22u
- R11, R9: value 1.5k -> NP_1k
- R3: value 22k -> 10k
- moved P2 0.15 mm to (61.5, 126.2)
Routing:
- net GND: track 217.4 -> 223.3 mm
- net Net-(BT1-Pad2): track 51.8 -> 52.9 mm
Other:
- rule pad_to_mask_clearance: 0.12 -> 0.1
- board text added: "+"
- board text added: "-"
- board text added: "SWADGE2019 REV C All Aircraft Report"
- board text removed: "SWADGE2019 REV B All Aircraft Report"
